Commit message: 整合

File: src/dual_arm_description/urdf/dual_arm.urdf.xacro (robot description, xacro)
@@ -2,8 +2,62 @@
 <robot xmlns:xacro="http://www.ros.org/wiki/xacro" name="dual_panda">
   <!-- ========================================================================= -->
-  <!-- 1. 定义一个纯净的手臂宏 (直接引用 Mesh，不依赖官方逻辑) -->
-  <!-- ========================================================================= -->
-  <xacro:macro name="clean_arm" params="arm_id connected_to xyz:='0 0 0' rpy:='0 0 0'">
-    <!-- 根关节 -->
+  <!-- 0. 基础宏定义 (物理修正版) -->
+  <!-- ========================================================================= -->
+  <xacro:macro name="cylinder_inertial" params="radius length mass *origin">
+    <inertial>
+      <mass value="${mass}" />
+      <xacro:insert_block name="origin" />
+      <inertia ixx="${0.0833333 * mass * (3 * radius * radius + length * length)}" ixy="0.0" ixz="0.0"
+               iyy="${0.0833333 * mass * (3 * radius * radius + length * length)}" iyz="0.0"
+               izz="${0.5 * mass * radius * radius}" />
+    </inertial>
+  </xacro:macro>
+  <xacro:macro name="box_inertial" params="x y z mass *origin">
+    <inertial>
+      <mass value="${mass}" />
+      <xacro:insert_block name="origin" />
+      <inertia ixx="${0.0833333 * mass * (y*y + z*z)}" ixy="0.0" ixz="0.0"
+               iyy="${0.0833333 * mass * (x*x + z*z)}" iyz="0.0"
+               izz="${0.0833333 * mass * (x*x + y*y)}" />
+    </inertial>
+  </xacro:macro>
+  <!-- [新增] 球体惯性宏，用于关节球 -->
+  <xacro:macro name="sphere_inertial" params="radius mass *origin">
+    <inertial>
+      <mass value="${mass}" />
+      <xacro:insert_block name="origin" />
+      <inertia ixx="${0.4 * mass * radius * radius}" ixy="0.0" ixz="0.0"
+               iyy="${0.4 * mass * radius * radius}" iyz="0.0"
+               izz="${0.4 * mass * radius * radius}" />
+    </inertial>
+  </xacro:macro>
+  <!-- 视觉宏：包含圆柱体体身 + 关节处的球体 -->
+  <xacro:macro name="visual_link_with_joint" params="radius length origin_xyz:='0 0 0' origin_rpy:='0 0 0'">
+     <!-- Link 本体 (圆柱) -->
+    <visual>
+      <origin xyz="${origin_xyz}" rpy="${origin_rpy}"/>
+      <geometry><cylinder radius="${radius}" length="${length}"/></geometry>
+      <material name="White"><color rgba="1 1 1 1"/></material>
+    </visual>
+    <!-- 关节球 (补缝) -->
+    <visual>
+      <origin xyz="0 0 0" rpy="0 0 0"/>
+      <geometry><sphere radius="${radius * 1.1}"/></geometry>
+      <material name="White"/>
+    </visual>
+  </xacro:macro>
+  <!-- [修正] 碰撞体宏：只保留圆柱，不包含关节球，防止运动卡死 -->
+  <xacro:macro name="simple_collision" params="radius length origin_xyz:='0 0 0' origin_rpy:='0 0 0'">
+    <collision>
+      <origin xyz="${origin_xyz}" rpy="${origin_rpy}"/>
+      <!-- 半径稍微缩小一点点，避免紧贴碰撞 -->
+      <geometry><cylinder radius="${radius * 0.9}" length="${length}"/></geometry>
+    </collision>
+  </xacro:macro>
+  <!-- ========================================================================= -->
+  <!-- 1. 机械臂宏 -->
+  <!-- ========================================================================= -->
+  <xacro:macro name="panda_arm" params="arm_id connected_to xyz:='0 0 0' rpy:='0 0 0'">
+    <!-- Base Link 固定关节 -->
     <joint name="${arm_id}_joint_base" type="fixed">
       <parent link="${connected_to}"/>
@@ -12,64 +66,99 @@
     </joint>
     <link name="${arm_id}_link0">
-      <visual><geometry><mesh filename="package://franka_description/meshes/robot_arms/fer/visual/link0.dae"/></geometry></visual>
-      <collision><geometry><mesh filename="package://franka_description/meshes/robot_arms/fer/collision/link0.stl"/></geometry></collision>
-    </link>
+      <xacro:visual_link_with_joint radius="0.06" length="0.1" origin_xyz="0 0 0.05" origin_rpy="0 0 0"/>
+      <xacro:simple_collision radius="0.06" length="0.1" origin_xyz="0 0 0.05"/>
+      <xacro:cylinder_inertial radius="0.06" length="0.1" mass="3.06"><origin xyz="0 0 0.05" rpy="0 0 0"/></xacro:cylinder_inertial>
+    </link>
+    <gazebo reference="${arm_id}_link0"><material>Gazebo/White</material></gazebo>
+    <joint name="${arm_id}_joint1" type="revolute">
+      <origin rpy="0 0 0" xyz="0 0 0.333"/> <parent link="${arm_id}_link0"/> <child link="${arm_id}_link1"/> <axis xyz="0 0 1"/>
+      <limit effort="87" lower="-2.8973" upper="2.8973" velocity="2.1750"/> <dynamics damping="1.0" friction="0.5"/>
+    </joint>
     <link name="${arm_id}_link1">
-      <visual><geometry><mesh filename="package://franka_description/meshes/robot_arms/fer/visual/link1.dae"/></geometry></visual>
-      <collision><geometry><mesh filename="package://franka_description/meshes/robot_arms/fer/collision/link1.stl"/></geometry></collision>
-    </link>
-    <joint name="${arm_id}_joint1" type="revolute">
-      <origin rpy="0 0 0" xyz="0 0 0.333"/> <parent link="${arm_id}_link0"/> <child link="${arm_id}_link1"/> <axis xyz="0 0 1"/> <limit effort="87" lower="-2.8973" upper="2.8973" velocity="2.1750"/>
+      <xacro:visual_link_with_joint radius="0.06" length="0.3" origin_xyz="0 0 -0.15"/>
+      <xacro:simple_collision radius="0.06" length="0.3" origin_xyz="0 0 -0.15"/>
+      <xacro:cylinder_inertial radius="0.06" length="0.3" mass="2.34"><origin xyz="0 0 -0.15" rpy="0 0 0"/></xacro:cylinder_inertial>
+    </link>
+    <gazebo reference="${arm_id}_link1"><material>Gazebo/White</material></gazebo>
+    <joint name="${arm_id}_joint2" type="revolute">
+      <origin rpy="${-pi/2} 0 0" xyz="0 0 0"/> <parent link="${arm_id}_link1"/> <child link="${arm_id}_link2"/> <axis xyz="0 0 1"/>
+      <limit effort="87" lower="-1.7628" upper="1.7628" velocity="2.1750"/> <dynamics damping="1.0" friction="0.5"/>
     </joint>
     <link name="${arm_id}_link2">
-      <visual><geometry><mesh filename="package://franka_description/meshes/robot_arms/fer/visual/link2.dae"/></geometry></visual>
-      <collision><geometry><mesh filename="package://franka_description/meshes/robot_arms/fer/collision/link2.stl"/></geometry></collision>
-    </link>
-    <joint name="${arm_id}_joint2" type="revolute">
-      <origin rpy="${-pi/2} 0 0" xyz="0 0 0"/> <parent link="${arm_id}_link1"/> <child link="${arm_id}_link2"/> <axis xyz="0 0 1"/> <limit effort="87" lower="-1.7628" upper="1.7628" velocity="2.1750"/>
+      <xacro:visual_link_with_joint radius="0.06" length="0.35" origin_xyz="0 -0.15 0" origin_rpy="-1.57 0 0"/>
+      <xacro:simple_collision radius="0.06" length="0.35" origin_xyz="0 -0.15 0" origin_rpy="-1.57 0 0"/>
+      <xacro:cylinder_inertial radius="0.06" length="0.35" mass="2.36"><origin xyz="0 -0.15 0" rpy="-1.57 0 0"/></xacro:cylinder_inertial>
+    </link>
+    <gazebo reference="${arm_id}_link2"><material>Gazebo/White</material></gazebo>
+    <joint name="${arm_id}_joint3" type="revolute">
+      <origin rpy="${pi/2} 0 0" xyz="0 -0.316 0"/> <parent link="${arm_id}_link2"/> <child link="${arm_id}_link3"/> <axis xyz="0 0 1"/>
+      <limit effort="87" lower="-2.8973" upper="2.8973" velocity="2.1750"/> <dynamics damping="1.0" friction="0.5"/>
     </joint>
     <link name="${arm_id}_link3">
-      <visual><geometry><mesh filename="package://franka_description/meshes/robot_arms/fer/visual/link3.dae"/></geometry></visual>
-      <collision><geometry><mesh filename="package://franka_description/meshes/robot_arms/fer/collision/link3.stl"/></geometry></collision>
-    </link>
-    <joint name="${arm_id}_joint3" type="revolute">
-      <origin rpy="${pi/2} 0 0" xyz="0 -0.316 0"/> <parent link="${arm_id}_link2"/> <child link="${arm_id}_link3"/> <axis xyz="0 0 1"/> <limit effort="87" lower="-2.8973" upper="2.8973" velocity="2.1750"/>
+       <xacro:visual_link_with_joint radius="0.06" length="0.2" origin_xyz="0 0 -0.1"/>
+       <xacro:simple_collision radius="0.06" length="0.2" origin_xyz="0 0 -0.1"/>
+      <xacro:cylinder_inertial radius="0.06" length="0.2" mass="2.38"><origin xyz="0 0 -0.1" rpy="0 0 0"/></xacro:cylinder_inertial>
+    </link>
+    <gazebo reference="${arm_id}_link3"><material>Gazebo/White</material></gazebo>
+    <joint name="${arm_id}_joint4" type="revolute">
+      <origin rpy="${pi/2} 0 0" xyz="0.0825 0 0"/> <parent link="${arm_id}_link3"/> <child link="${arm_id}_link4"/> <axis xyz="0 0 1"/>
+      <limit effort="87" lower="-3.0718" upper="-0.0698" velocity="2.1750"/> <dynamics damping="1.0" friction="0.5"/>
     </joint>
     <link name="${arm_id}_link4">
-      <visual><geometry><mesh filename="package://franka_description/meshes/robot_arms/fer/visual/link4.dae"/></geometry></visual>
-      <collision><geometry><mesh filename="package://franka_description/meshes/robot_arms/fer/collision/link4.stl"/></geometry></collision>
-    </link>
-    <joint name="${arm_id}_joint4" type="revolute">
-      <origin rpy="${pi/2} 0 0" xyz="0.0825 0 0"/> <parent link="${arm_id}_link3"/> <child link="${arm_id}_link4"/> <axis xyz="0 0 1"/> <limit effort="87" lower="-3.0718" upper="-0.0698" velocity="2.1750"/>
+       <xacro:visual_link_with_joint radius="0.06" length="0.2" origin_xyz="0 0.1 0" origin_rpy="1.57 0 0"/>
+       <xacro:simple_collision radius="0.06" length="0.2" origin_xyz="0 0.1 0" origin_rpy="1.57 0 0"/>
+      <xacro:cylinder_inertial radius="0.06" length="0.2" mass="2.43"><origin xyz="0 0 0" rpy="0 0 0"/></xacro:cylinder_inertial>
+    </link>
+    <gazebo reference="${arm_id}_link4"><material>Gazebo/White</material></gazebo>
+    <joint name="${arm_id}_joint5" type="revolute">
+      <origin rpy="${-pi/2} 0 0" xyz="-0.0825 0.384 0"/> <parent link="${arm_id}_link4"/> <child link="${arm_id}_link5"/> <axis xyz="0 0 1"/>
+      <limit effort="12" lower="-2.8973" upper="2.8973" velocity="2.6100"/> <dynamics damping="1.0" friction="0.5"/>
     </joint>
     <link name="${arm_id}_link5">
-      <visual><geometry><mesh filename="package://franka_description/meshes/robot_arms/fer/visual/link5.dae"/></geometry></visual>
-      <collision><geometry><mesh filename="package://franka_description/meshes/robot_arms/fer/collision/link5.stl"/></geometry></collision>
-    </link>
-    <joint name="${arm_id}_joint5" type="revolute">
-      <origin rpy="${-pi/2} 0 0" xyz="-0.0825 0.384 0"/> <parent link="${arm_id}_link4"/> <child link="${arm_id}_link5"/> <axis xyz="0 0 1"/> <limit effort="12" lower="-2.8973" upper="2.8973" velocity="2.6100"/>
+       <xacro:visual_link_with_joint radius="0.05" length="0.25" origin_xyz="0 0 -0.125"/>
+       <xacro:simple_collision radius="0.05" length="0.25" origin_xyz="0 0 -0.125"/>
+      <xacro:cylinder_inertial radius="0.05" length="0.25" mass="3.5"><origin xyz="0 0 -0.125" rpy="0 0 0"/></xacro:cylinder_inertial>
+    </link>
+    <gazebo reference="${arm_id}_link5"><material>Gazebo/White</material></gazebo>
+    <joint name="${arm_id}_joint6" type="revolute">
+      <origin rpy="${pi/2} 0 0" xyz="0 0 0"/> <parent link="${arm_id}_link5"/> <child link="${arm_id}_link6"/> <axis xyz="0 0 1"/>
+      <limit effort="12" lower="-0.0175" upper="3.7525" velocity="2.6100"/> <dynamics damping="0.5" friction="0.5"/>
     </joint>
     <link name="${arm_id}_link6">
-      <visual><geometry><mesh filename="package://franka_description/meshes/robot_arms/fer/visual/link6.dae"/></geometry></visual>
-      <collision><geometry><mesh filename="package://franka_description/meshes/robot_arms/fer/collision/link6.stl"/></geometry></collision>
-    </link>
-    <joint name="${arm_id}_joint6" type="revolute">
-      <origin rpy="${pi/2} 0 0" xyz="0 0 0"/> <parent link="${arm_id}_link5"/> <child link="${arm_id}_link6"/> <axis xyz="0 0 1"/> <limit effort="12" lower="0.0175" upper="3.7525" velocity="2.6100"/>
+       <xacro:visual_link_with_joint radius="0.05" length="0.1" origin_xyz="0 0 0"/>
+       <xacro:simple_collision radius="0.05" length="0.1" origin_xyz="0 0 0"/>
+      <xacro:cylinder_inertial radius="0.05" length="0.1" mass="1.47"><origin xyz="0 0 0" rpy="0 0 0"/></xacro:cylinder_inertial>
+    </link>
+    <gazebo reference="${arm_id}_link6"><material>Gazebo/White</material></gazebo>
+    <joint name="${arm_id}_joint7" type="revolute">
+      <origin rpy="${pi/2} 0 0" xyz="0.088 0 0"/> <parent link="${arm_id}_link6"/> <child link="${arm_id}_link7"/> <axis xyz="0 0 1"/>
+      <limit effort="12" lower="-2.8973" upper="2.8973" velocity="2.6100"/> <dynamics damping="0.5" friction="0.5"/>
     </joint>
     <link name="${arm_id}_link7">
-      <visual><geometry><mesh filename="package://franka_description/meshes/robot_arms/fer/visual/link7.dae"/></geometry></visual>
-      <collision><geometry><mesh filename="package://franka_description/meshes/robot_arms/fer/collision/link7.stl"/></geometry></collision>
-    </link>
-    <joint name="${arm_id}_joint7" type="revolute">
-      <origin rpy="${pi/2} 0 0" xyz="0.088 0 0"/> <parent link="${arm_id}_link6"/> <child link="${arm_id}_link7"/> <axis xyz="0 0 1"/> <limit effort="12" lower="-2.8973" upper="2.8973" velocity="2.6100"/>
-    </joint>
-    <link name="${arm_id}_link8"/>
+       <xacro:visual_link_with_joint radius="0.04" length="0.08" origin_xyz="0 0 0.04"/>
+       <xacro:simple_collision radius="0.04" length="0.08" origin_xyz="0 0 0.04"/>
+      <xacro:cylinder_inertial radius="0.04" length="0.08" mass="0.45"><origin xyz="0 0 0.04" rpy="0 0 0"/></xacro:cylinder_inertial>
+    </link>
+    <gazebo reference="${arm_id}_link7"><material>Gazebo/White</material></gazebo>
     <joint name="${arm_id}_joint8" type="fixed">
       <origin rpy="0 0 0" xyz="0 0 0.107"/> <parent link="${arm_id}_link7"/> <child link="${arm_id}_link8"/>
     </joint>
-  </xacro:macro>
-<!-- 2. 夹爪宏 (修改版：修复闪退 + 可活动的关节) -->
-  <xacro:macro name="simple_hand" params="arm_id connected_to rpy:='0 0 0' xyz:='0 0 0'">
-    <!-- 手掌基座 -->
+    <link name="${arm_id}_link8">
+      <visual>
+        <!-- 保持原点，不需要偏移，连接关节已经偏移过了 -->
+        <geometry><cylinder radius="0.04" length="0.04"/></geometry>
+        <material name="Grey"><color rgba="0.5 0.5 0.5 1"/></material>
+      </visual>
+      <collision>
+          <geometry><cylinder radius="0.04" length="0.04"/></geometry>
+      </collision>
+      <xacro:cylinder_inertial radius="0.04" length="0.04" mass="0.1"><origin xyz="0 0 0" rpy="0 0 0"/></xacro:cylinder_inertial>
+    </link>
+    <gazebo reference="${arm_id}_link8"><material>Gazebo/Grey</material></gazebo>
+  </xacro:macro>
+  <!-- ========================================================================= -->
+  <!-- 2. 手部宏 (物理修正) -->
+  <!-- ========================================================================= -->
+  <xacro:macro name="panda_hand" params="arm_id connected_to rpy:='0 0 0' xyz:='0 0 0'">
     <joint name="${arm_id}_hand_joint" type="fixed">
       <parent link="${connected_to}"/>
@@ -78,67 +167,109 @@
     </joint>
     <link name="${arm_id}_hand">
-      <visual><geometry><mesh filename="package://franka_description/meshes/robot_ee/franka_hand_white/visual/hand.dae"/></geometry></visual>
-      <!-- 如果之后运行手掌(hand)也报错找不到文件，请把下面这行的 collision/hand.stl 也改成 visual/hand.dae -->
-      <collision><geometry><mesh filename="package://franka_description/meshes/robot_ee/franka_hand_white/collision/hand.stl"/></geometry></collision>
-    </link>
-    <!-- 左指头 -->
+      <visual>
+          <origin xyz="0 0 0.04" rpy="0 0 0"/>
+          <geometry><box size="0.1 0.06 0.08"/></geometry>
+          <material name="Grey"><color rgba="0.5 0.5 0.5 1"/></material>
+      </visual>
+      <!-- [修正] 缩小 Collision 尺寸，防止与手指互相弹开 -->
+      <collision>
+        <origin xyz="0 0 0.04" rpy="0 0 0"/>
+        <geometry><box size="0.08 0.05 0.06"/></geometry>
+      </collision>
+      <xacro:box_inertial x="0.1" y="0.1" z="0.1" mass="0.6"><origin xyz="0 0 0" rpy="0 0 0"/></xacro:box_inertial>
+    </link>
+    <gazebo reference="${arm_id}_hand"><material>Gazebo/Grey</material></gazebo>
     <link name="${arm_id}_leftfinger">
-       <visual><origin xyz="0 -0.007 0" rpy="0 0 ${pi}"/><geometry><mesh filename="package://franka_description/meshes/robot_ee/franka_hand_white/visual/finger.dae"/></geometry></visual>
-       <collision><origin xyz="0 -0.007 0" rpy="0 0 ${pi}"/><geometry><mesh filename="package://franka_description/meshes/robot_ee/franka_hand_white/visual/finger.dae"/></geometry></collision>
-    </link>
-    <!-- 右指头 -->
+      <visual>
+          <origin xyz="0 0.015 0.03" rpy="0 0 0"/>
+          <geometry><box size="0.022 0.022 0.04"/></geometry>
+          <material name="Grey"><color rgba="0.5 0.5 0.5 1"/></material>
+      </visual>
+      <!-- [修正] 缩小碰撞体，稍微远离中心 -->
+      <collision><origin xyz="0 0.015 0.03" rpy="0 0 0"/><geometry><box size="0.015 0.015 0.03"/></geometry></collision>
+      <xacro:box_inertial x="0.02" y="0.02" z="0.05" mass="0.1"><origin xyz="0 0 0" rpy="0 0 0"/></xacro:box_inertial>
+    </link>
+    <gazebo reference="${arm_id}_leftfinger"><material>Gazebo/Grey</material></gazebo>
+    <joint name="${arm_id}_finger_joint1" type="prismatic">
+      <parent link="${arm_id}_hand"/> <child link="${arm_id}_leftfinger"/> <origin xyz="0 0 0.0584" rpy="0 0 0"/> <axis xyz="0 1 0"/>
+      <limit effort="20" lower="0.0" upper="0.04" velocity="0.2"/> <dynamics damping="0.1" friction="0.1"/>
+    </joint>
     <link name="${arm_id}_rightfinger">
-      <visual><origin xyz="0 0.007 0" rpy="0 0 0"/><geometry><mesh filename="package://franka_description/meshes/robot_ee/franka_hand_white/visual/finger.dae"/></geometry></visual>
-      <collision><origin xyz="0 0.007 0" rpy="0 0 0"/><geometry><mesh filename="package://franka_description/meshes/robot_ee/franka_hand_white/visual/finger.dae"/></geometry></collision>
-    </link>
-    <!-- 关节定义 (保持之前的 prismatic 改动) -->
-    <joint name="${arm_id}_finger_joint1" type="prismatic">
-      <parent link="${arm_id}_hand"/>
-      <child link="${arm_id}_leftfinger"/>
-      <origin xyz="0 0 0.0584" rpy="0 0 0"/>
-      <axis xyz="0 1 0"/> <!-- 沿 Y 轴滑动 -->
-      <limit effort="20" lower="0.0" upper="0.09" velocity="0.2"/>
-    </joint>
+      <visual>
+          <origin xyz="0 -0.015 0.03" rpy="0 0 0"/>
+          <geometry><box size="0.022 0.022 0.04"/></geometry>
+          <material name="Grey"><color rgba="0.5 0.5 0.5 1"/></material>
+      </visual>
+      <!-- [修正] 缩小碰撞体 -->
+      <collision><origin xyz="0 -0.015 0.03" rpy="0 0 0"/><geometry><box size="0.015 0.015 0.03"/></geometry></collision>
+      <xacro:box_inertial x="0.02" y="0.02" z="0.05" mass="0.1"><origin xyz="0 0 0" rpy="0 0 0"/></xacro:box_inertial>
+    </link>
+    <gazebo reference="${arm_id}_rightfinger"><material>Gazebo/Grey</material></gazebo>
     <joint name="${arm_id}_finger_joint2" type="prismatic">
-      <parent link="${arm_id}_hand"/>
-      <child link="${arm_id}_rightfinger"/>
-      <origin xyz="0 0 0.0584" rpy="0 0 0"/>
-      <axis xyz="0 1 0"/> <!-- 沿 Y 轴滑动 -->
-      <limit effort="20" lower="0.0" upper="0.09" velocity="0.2"/>
-    </joint>
-  </xacro:macro>
-  <!-- ========================================================================= -->
-  <!-- 3. 实例化：根连杆 base_link -->
-  <!-- ========================================================================= -->
-  <link name="base_link"/>
-  <!-- 左臂 -->
-  <xacro:clean_arm arm_id="panda_1" connected_to="base_link" xyz="-0.5 0 0" rpy="0 0 0"/>
-  <xacro:simple_hand arm_id="panda_1" connected_to="panda_1_link8" rpy="0 0 ${-pi/4}"/>
-  <!-- 右臂 -->
-  <xacro:clean_arm arm_id="panda_2" connected_to="base_link" xyz="0.5 0 0" rpy="0 0 ${pi}"/>
-  <xacro:simple_hand arm_id="panda_2" connected_to="panda_2_link8" rpy="0 0 ${-pi/4}"/>
-  <!-- ========================================================================= -->
-  <!-- 4. 硬件接口 (必不可少) -->
-  <!-- ========================================================================= -->
-  <ros2_control name="DualPandaFakeSystem" type="system">
-    <hardware><plugin>mock_components/GenericSystem</plugin></hardware>
-    <xacro:macro name="config_joint" params="name">
-      <joint name="${name}">
-        <command_interface name="position"/><state_interface name="position"><param name="initial_value">0.0</param></state_interface><state_interface name="velocity"/>
-      </joint>
+      <parent link="${arm_id}_hand"/> <child link="${arm_id}_rightfinger"/> <origin xyz="0 0 0.0584" rpy="0 0 0"/> <axis xyz="0 -1 0"/>
+      <limit effort="20" lower="0.0" upper="0.04" velocity="0.2"/> <dynamics damping="0.1" friction="0.1"/>
+      <mimic joint="${arm_id}_finger_joint1" multiplier="1" offset="0"/>
+    </joint>
+  </xacro:macro>
+  <!-- ========================================================================= -->
+  <!-- 3. 场景构建 -->
+  <!-- ========================================================================= -->
+  <link name="world"/>
+  <joint name="world_joint" type="fixed">
+    <parent link="world"/>
+    <child link="base_link"/>
+    <origin xyz="0 0 0.05" rpy="0 0 0"/>
+  </joint>
+  <link name="base_link">
+    <visual><geometry><box size="0.4 1.2 0.1"/></geometry><material name="Gray"><color rgba="0.6 0.6 0.6 1"/></material></visual>
+    <collision><geometry><box size="0.4 1.2 0.1"/></geometry></collision>
+    <xacro:box_inertial x="0.4" y="1.2" z="0.1" mass="100.0"><origin xyz="0 0 0" rpy="0 0 0"/></xacro:box_inertial>
+  </link>
+  <gazebo reference="base_link"> <material>Gazebo/Gray</material> </gazebo>
+  <xacro:panda_arm arm_id="panda_1" connected_to="base_link" xyz="0 -0.4 0.05" rpy="0 0 0"/>
+  <xacro:panda_hand arm_id="panda_1" connected_to="panda_1_link8" rpy="0 0 ${-pi/4}"/>
+  <xacro:panda_arm arm_id="panda_2" connected_to="base_link" xyz="0 0.4 0.05" rpy="0 0 0"/>
+  <xacro:panda_hand arm_id="panda_2" connected_to="panda_2_link8" rpy="0 0 ${-pi/4}"/>
+  <!-- ROS2 Control (保持不变) -->
+  <ros2_control name="GazeboSystem" type="system">
+    <hardware><plugin>gazebo_ros2_control/GazeboSystem</plugin></hardware>
+    <xacro:macro name="config_joint" params="name initial_pos">
+        <joint name="${name}">
+            <command_interface name="position"/>
+            <state_interface name="position"><param name="initial_value">${initial_pos}</param></state_interface>
+            <state_interface name="velocity"/>
+        </joint>
     </xacro:macro>
-    <xacro:config_joint name="panda_1_joint1"/> <xacro:config_joint name="panda_1_joint2"/>
-    <xacro:config_joint name="panda_1_joint3"/> <xacro:config_joint name="panda_1_joint4"/>
-    <xacro:config_joint name="panda_1_joint5"/> <xacro:config_joint name="panda_1_joint6"/>
-    <xacro:config_joint name="panda_1_joint7"/>
-    <xacro:config_joint name="panda_2_joint1"/> <xacro:config_joint name="panda_2_joint2"/>
-    <xacro:config_joint name="panda_2_joint3"/> <xacro:config_joint name="panda_2_joint4"/>
-    <xacro:config_joint name="panda_2_joint5"/> <xacro:config_joint name="panda_2_joint6"/>
-    <xacro:config_joint name="panda_2_joint7"/>
-    <!-- 增加夹爪关节配置 -->
-    <xacro:config_joint name="panda_1_finger_joint1"/>
-    <xacro:config_joint name="panda_1_finger_joint2"/>
-    <xacro:config_joint name="panda_2_finger_joint1"/>
-    <xacro:config_joint name="panda_2_finger_joint2"/>
+    <xacro:config_joint name="panda_1_joint1" initial_pos="0.0"/>
+    <xacro:config_joint name="panda_1_joint2" initial_pos="-0.785"/>
+    <xacro:config_joint name="panda_1_joint3" initial_pos="0.0"/>
+    <xacro:config_joint name="panda_1_joint4" initial_pos="-2.356"/>
+    <xacro:config_joint name="panda_1_joint5" initial_pos="0.0"/>
+    <xacro:config_joint name="panda_1_joint6" initial_pos="1.571"/>
+    <xacro:config_joint name="panda_1_joint7" initial_pos="0.785"/>
+    <xacro:config_joint name="panda_2_joint1" initial_pos="0.0"/>
+    <xacro:config_joint name="panda_2_joint2" initial_pos="-0.785"/>
+    <xacro:config_joint name="panda_2_joint3" initial_pos="0.0"/>
+    <xacro:config_joint name="panda_2_joint4" initial_pos="-2.356"/>
+    <xacro:config_joint name="panda_2_joint5" initial_pos="0.0"/>
+    <xacro:config_joint name="panda_2_joint6" initial_pos="1.571"/>
+    <xacro:config_joint name="panda_2_joint7" initial_pos="0.785"/>
+    <xacro:config_joint name="panda_1_finger_joint1" initial_pos="0.0"/>
+    <!-- <xacro:config_joint name="panda_1_finger_joint2" initial_pos="0.0"/> -->
+    <xacro:config_joint name="panda_2_finger_joint1" initial_pos="0.0"/>
+    <!-- <xacro:config_joint name="panda_2_finger_joint2" initial_pos="0.0"/> -->
+    <!-- [关键修复] 为模仿关节（Mimic Joints）添加被动接口，防止 Gazebo 崩溃 -->
+    <!-- 注意：不要给 mimic joint 添加 command_interface，但需要这一块占位符或者完全移除 ros2_control标签 -->
+    <!-- 最佳实践：在 gazebo_ros2_control 中，mimic 关节通常不需要显式定义 command_interface -->
+    <!-- 如果定义了，必须由 mimic 插件接管，或者通过 controller 驱动。这里我们在 URDF 层面让其被动。-->
   </ros2_control>
+  <gazebo>
+    <plugin filename="libgazebo_ros2_control.so" name="gazebo_ros2_control">
+      <parameters>$(find dual_arm_moveit_config)/config/ros2_controllers.yaml</parameters>
+      <!-- [关键修复] 显式告知插件处理 mimic 关节 -->
+      <ros>
+        <namespace>/</namespace>
+      </ros>
+    </plugin>
+  </gazebo>
 </robot>
